Commit message: added dummy urdf visuals

File: bot_desc/urdf/bot_orig.urdf.xacro (robot description, xacro)
@@ -14,13 +14,13 @@
     <link name="base_cone">
         <visual>
-            <origin xyz="0.0 0.0 0.0375" rpy="0.0 0.0 0.0"/>
-            <geometry>
-                <cylinder radius="0.05" length="0.075"/>
-            </geometry>
-        </visual>
-        <collision>
-            <origin xyz="0.0 0.0 0.0375" rpy="0.0 0.0 0.0"/>
-            <geometry>
-                <cylinder radius="0.05" length="0.075"/>
+            <origin xyz="0.0 0.0 0.0" rpy="0.0 0.0 0.0"/>
+            <geometry>
+                <mesh filename="package://bot_desc/meshes/new_base_cone.stl" scale="0.001 0.001 0.001"/>
+            </geometry>
+        </visual>
+        <collision>
+            <origin xyz="0.0 0.0 0.0" rpy="0.0 0.0 0.0"/>
+            <geometry>
+                <mesh filename="package://bot_desc/meshes/new_base_cone.stl" scale="0.001 0.001 0.001"/>
             </geometry>
         </collision>
@@ -59,7 +59,7 @@
     <link name="shoulder_motor">
         <visual>
-            <origin xyz="0.0 0.0 0.0375" rpy="0.0 0.0 0.0"/>
-            <geometry>
-                <box size="0.05 0.050 0.075"/>
+            <origin xyz="0.0 0.0 -0.0775" rpy="0.0 0.0 0.0"/>
+            <geometry>
+                <mesh filename="package://bot_desc/meshes/shoulder_motor.stl" />
             </geometry>
             <material name="blue">
@@ -68,7 +68,7 @@
         </visual>
         <collision>
-            <origin xyz="0.0 0.0 0.03750" rpy="0.0 0.0 0.0"/>
-            <geometry>
-                <box size="0.05 0.050 0.075"/>
+            <origin xyz="0.0 0.0 -0.0775" rpy="0.0 0.0 0.0"/>
+            <geometry>
+                <mesh filename="package://bot_desc/meshes/shoulder_motor.stl" />
             </geometry>
         </collision>
@@ -82,7 +82,7 @@
     <link name="shoulder_arm">
         <visual>
-            <origin xyz="0.0 0.0 0.05" rpy="0.0 0.0 0.0"/>
-            <geometry>
-                <box size="0.04 0.04 0.1"/>
+            <origin xyz="0.0 0.0 -0.1375" rpy="0.0 0.0 0.0"/>
+            <geometry>
+                <mesh filename="package://bot_desc/meshes/shoulder_arm.stl" />
             </geometry>
             <material name="red_material">
@@ -91,7 +91,7 @@
         </visual>
         <collision>
-            <origin xyz="0.0 0.0 0.05" rpy="0.0 0.0 0.0"/>
-            <geometry>
-                <box size="0.04 0.04 0.1"/>
+            <origin xyz="0.0 0.0 -0.1375" rpy="0.0 0.0 0.0"/>
+            <geometry>
+                <mesh filename="package://bot_desc/meshes/shoulder_arm.stl" />
             </geometry>
         </collision>
@@ -99,5 +99,5 @@
     </link>
     <joint name="shoulder_motor_to_shoulder_arm" type="revolute">
-        <origin xyz="0.0 0.0 0.075" rpy="0.0 0.0 0.0"/>
+        <origin xyz="0.0 0.0 0.06" rpy="0.0 0.0 0.0"/>
         <parent link="shoulder_motor"/>
         <child link="shoulder_arm"/>
@@ -107,8 +107,7 @@
     <link name="elbow_arm">
         <visual>
-            <origin xyz="0.0 0.0 0.04" rpy="0.0 0.0 0.0"/>
-            <geometry>
-                <!-- <cylinder radius="0.03" length="0.08"/> -->
-                <box size="0.03 0.03 0.08"/>
+            <origin xyz="0.0 0.0 -0.3225" rpy="0.0 0.0 0.0"/>
+            <geometry>
+                <mesh filename="package://bot_desc/meshes/elbow_arm.stl"/>
             </geometry>
             <material name="elbow_arm_material">
@@ -117,7 +116,7 @@
         </visual>
         <collision>
-            <origin xyz="0.0 0.0 0.04" rpy="0.0 0.0 0.0"/>
-            <geometry>
-                <box size="0.03 0.03 0.08"/>
+            <origin xyz="0.0 0.0 -0.3275" rpy="0.0 0.0 0.0"/>
+            <geometry>
+                <mesh filename="package://bot_desc/meshes/elbow_arm.stl"/>
             </geometry>
         </collision>
@@ -125,5 +124,5 @@
     </link>
     <joint name="shoulder_to_elbow" type="revolute">
-        <origin xyz="0.0 0.0 0.1" rpy="0.0 0.0 0.0"/>
+        <origin xyz="0.0 0.0 0.185" rpy="0.0 0.0 0.0"/>
         <parent link="shoulder_arm"/>
         <child link="elbow_arm"/>
@@ -150,5 +149,5 @@
     </link>
     <joint name="elbow_to_wrist_attachment" type="revolute">
-        <origin xyz="0.0 0.0 0.08" rpy="0.0 0.0 0.0"/>
+        <origin xyz="0.0 0.0 0.132" rpy="0.0 0.0 0.0"/>
         <parent link="elbow_arm"/>
         <child link="wrist_attachment_1"/>
@@ -158,5 +157,5 @@
     <link name='utensil_attachment'>
         <visual>
-            <origin xyz="-0.04 -0.03625 -0.46" rpy="0.0 0.0 0.0"/>
+            <origin xyz="-0.04 -0.03825 -0.4625" rpy="0.0 0.0 0.0"/>
             <geometry>
                 <mesh filename="package://bot_desc/meshes/utensil_attachment.stl"/>
@@ -167,5 +166,5 @@
         </visual>
         <collision>
-            <origin xyz="-0.04 -0.03625 -0.46" rpy="0.0 0.0 0.0"/>
+            <origin xyz="-0.04 -0.03825 -0.4625" rpy="0.0 0.0 0.0"/>
             <geometry>
                 <mesh filename="package://bot_desc/meshes/utensil_attachment.stl"/>
@@ -199,6 +198,6 @@
         <xacro:default_inertial mass="1.0"/>
     </link>
-    <joint name="utensil_to_handle" type="fixed">
-        <origin xyz="0.0 0.1 -0.018" rpy="0.0 0.0 0.0"/>
+    <joint name="utensil_to_spatula" type="fixed">
+        <origin xyz="0.0425 -0.6 0.5" rpy="0.0 0.0 0.0"/>
         <parent link="utensil_attachment"/>
         <child link="handle"/>
@@ -222,6 +221,6 @@
         <xacro:default_inertial mass="1.0"/>
     </link>
-    <joint name="handle_to_spatula" type="fixed">
-        <origin xyz="0.0 0.0 0.0" rpy="0.0 0.0 0.0"/>
+    <joint name="spatula_to_handle" type="fixed">
+        <origin xyz="0.0 -0.2 0.0" rpy="0.0 0.0 0.0"/>
         <parent link="handle"/>
         <child link="spatula"/>
@@ -229,15 +228,15 @@
     <link name="grill">
         <visual name="">
-            <origin xyz="0 0.125 0.05" rpy="0.0 0.0 0.0"/>
+            <origin xyz="0 0.125 0.0" rpy="0.0 0.0 0.0"/>
             <geometry>
                 <box size="0.500 0.250 0.1"/>
             </geometry>
             <material name="">
-                <color rgba="0.0 1.0 0.0 1.0"/>
+                <color rgba="1.0 0.0 0.0 1.0"/>
                 <texture filename=""/>
             </material>
         </visual>
         <collision>
-            <origin xyz="0 0.125 0.0" rpy="0.0 0.0 0.0"/>
+            <origin xyz="0 0 0.0" rpy="0.0 0.0 0.0"/>
             <geometry>
                 <box size="0.500 0.250 0.0"/>
@@ -247,5 +246,5 @@
     </link>
     <joint name="grill_to_world" type="fixed">
-        <origin xyz="0 0.25 0.0" rpy="0.0 0.0 0.0"/>
+        <origin xyz="0 0.0500 0.0" rpy="0.0 0.0 0.0"/>
         <parent link="world"/>
         <child link="grill"/>
