Commit message: added burger cyl

File: bot_desc/urdf/bot.urdf.xacro (robot description, xacro)
@@ -7,5 +7,5 @@
         <inertial>
             <origin xyz="0.0 0.0 0.0" rpy="0.0 0.0 0.0"/>
-            <mass value="${mass}"/>
+            <mass value="${mass}" unit="kg"/>
             <inertia ixx="1.0" ixy="0.0" ixz="0.0" iyy="1.0" iyz="0.0" izz="1.0"/>
         </inertial>
@@ -227,4 +227,27 @@
         <child link="spatula"/>
     </joint>
+    <link name="burger">
+        <visual name="">
+            <origin xyz="0.0 0.0 0.05" rpy="0.0 0.0 0.0"/>
+            <geometry>
+                <cylinder radius="0.05" length="0.1"/>
+            </geometry>
+            <material name="">
+                <color rgba="1.0 1.0 1.0 1.0"/>
+            </material>
+        </visual>
+        <collision>
+            <origin xyz="0.0 0.0 0.05" rpy="0.0 0.0 0.0"/>
+            <geometry>
+                <cylinder radius="0.05" length="0.1"/>
+            </geometry>
+        </collision>
+        <xacro:default_inertial mass="1.0"/>
+    </link>
+    <joint name="spatula_to_burger" type="fixed">
+        <origin xyz="0.0 0.02 0.005" rpy="0.0 0.0 0.0"/>
+        <parent link="spatula"/>
+        <child link="burger"/>
+    </joint>
     <link name="grill">
         <visual name="">

Commit message: added effort and velocity

File: bot_desc/urdf/bot.urdf.xacro (robot description, xacro)
@@ -129,5 +129,5 @@
         <child link="elbow_arm"/>
         <axis xyz="1.0 0.0 0.0"/>
-        <limit lower="-1.57" upper="1.57" effort="0.0" velocity="0.0"/>
+        <limit lower="-1.57" upper="1.57" effort="1.962" velocity="5.236"/>
     </joint>
     <link name="wrist_attachment_1">
@@ -154,5 +154,5 @@
         <child link="wrist_attachment_1"/>
         <axis xyz="1.0 0.0 0.0"/>
-        <limit lower="-2.75" upper="2.75" effort="0.0" velocity="0.0"/>
+        <limit lower="-2.75" upper="2.75" effort="1.3734" velocity="10.472"/>
     </joint>
     <link name='utensil_attachment'>
@@ -243,5 +243,5 @@
             </geometry>
         </collision>
-        <xacro:default_inertial mass="1.0"/>
+        <xacro:default_inertial mass="10.0"/>
     </link>
     <joint name="spatula_to_burger" type="fixed">

Commit message: added setPoseTarget but has issues

File: bot_desc/urdf/bot.urdf.xacro (robot description, xacro)
@@ -55,5 +55,5 @@
         <child link="shoulder_attachment"/>
         <axis xyz="0.0 0.0 1.0"/>
-        <limit lower="-1.57" upper="1.57" effort="0.0" velocity="0.0"/>
+        <limit lower="-1.57" upper="1.57" effort="1.3734" velocity="10.0"/>
     </joint>
     <link name="shoulder_motor">
@@ -103,5 +103,5 @@
         <child link="shoulder_arm"/>
         <axis xyz="1.0 0.0 0.0"/>
-        <limit lower="-1.57" upper="1.57" effort="0.0" velocity="0.0"/>
+        <limit lower="-1.57" upper="1.57" effort="7.848" velocity="5.527"/>
     </joint>
     <link name="elbow_arm">
@@ -179,5 +179,5 @@
         <child link="utensil_attachment"/>
         <axis xyz="0.0 1.0 0.0"/>
-        <limit lower="-3.14" upper="3.14" effort="0.0" velocity="0.0"/>
+        <limit lower="-3.14" upper="3.14" effort="1.3734" velocity="10.0"/>
     </joint>
     <link name='handle'>
